Commit message: Fixed base gripper model path issue

File: models/base_gripper_model.urdf (robot description, URDF)
Before this commit: robot gripper, 2 links, 1 joints
Links:
- added link left_gripper_link; collision box size=0.01 0.032 0.04; visual box size=0.01 0.032 0.04
- added link right_gripper_link; collision box size=0.01 0.032 0.04; visual box size=0.01 0.032 0.04
Joints:
- added joint left_gripper_base_joint: type prismatic, parent base_link, child left_gripper_link, origin xyz=-0.054 0.0 -0.0555 rpy=0.0 0.0 0.0, axis 1.0 0.0 0.0, limit lower=0.0 upper=0.049 effort=100.0 velocity=1.0
- added joint right_gripper_base_joint: type prismatic, parent base_link, child right_gripper_link, origin xyz=0.054 0.0 -0.0555 rpy=0.0 0.0 0.0, axis 1.0 0.0 0.0, limit lower=-0.049 upper=0.0 effort=100.0 velocity=1.0
- joint base_joint: axis (none) -> 0.0 0.0 1.0; limit (none) -> lower=-0.3 upper=0 effort=100.0 velocity=1.0; origin (none) -> xyz=0.0 0.0 0.1 rpy=0.0 0.0 0.0; type fixed -> prismatic

Commit message: set init and target z position based on bounding box, updated gripper URDF Z limit

File: models/base_gripper_model.urdf (robot description, URDF)
Before this commit: robot gripper, 4 links, 3 joints
Joints:
- joint base_joint: limit lower=-0.3 upper=0 effort=100.0 velocity=1.0 -> lower=-0.3 upper=0.3 effort=100.0 velocity=1.0
